File: Circuits/PCB_design.kicad_sch (KiCad schematic)
At the start: 21 parts, among them J1 Inputs of IR sensors, J2 Battery, J3 Motors, J4 Sonar, U1 ATmega168A-P, U2 L293D, U3 L7805CV

Commit message: Update
Connections:
- net LED_1HZ: now also U1.9 (XTAL1/PB6)
- net LED_Sonar: now also U1.13 (PD7); no longer U1.23 (PC0)
Changed lines of the file:
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@@
+    )
+  )
+  (global_label "LED_1HZ" (shape input) (at 58.42 55.88 0) (fields_autoplaced)
+    (effects (font (size 1.27 1.27)) (justify left))
+    (property "Intersheet References" "${INTERSHEET_REFS}" (id 0) (at 68.9974 55.8006 0)
+      (effects (font (size 1.27 1.27)) (justify left) hide)
     )
   )
@@
     )
   )
-  (global_label "LED_Sonar" (shape input) (at 58.42 63.5 0) (fields_autoplaced)
+  (global_label "LED_Sonar" (shape input) (at 58.42 101.6 0) (fields_autoplaced)
     (effects (font (size 1.27 1.27)) (justify left))
-    (property "Intersheet References" "${INTERSHEET_REFS}" (id 0) (at 70.6907 63.4206 0)
+    (property "Intersheet References" "${INTERSHEET_REFS}" (id 0) (at 70.6907 101.5206 0)
       (effects (font (size 1.27 1.27)) (justify left) hide)
     )
